Commit message: Linorobot2 Gazebo Fortress - Harmonic

File: linorobot2_description/urdf/2wd_properties.urdf.xacro (robot description, xacro)
@@ -8,5 +8,5 @@
   <xacro:property name="wheel_width" value="0.01" />
   <xacro:property name="wheel_pos_x" value="0.0" />
-  <xacro:property name="wheel_pos_y" value="0.13" />
+  <xacro:property name="wheel_pos_y" value="0.145" />
   <xacro:property name="wheel_pos_z" value="-0.03" />
   <xacro:property name="wheel_mass" value=".1" />

File: linorobot2_description/urdf/controllers/diff_drive.urdf.xacro (robot description, xacro)
@@ -1,21 +1,22 @@
 <robot xmlns:xacro="http://ros.org/wiki/xacro">
-  <xacro:macro name="diff_drive_controller" params="wheel_separation wheel_radius wheel_torque">
+  <xacro:macro name="diff_drive_controller" params="wheel_separation wheel_radius">
     <gazebo>
-      <plugin name="differential_drive_controller" filename="libgazebo_ros_diff_drive.so">
-        <ros>
-          <remapping>odom:=odom/unfiltered</remapping>
-        </ros>
-        <updateRate>100</updateRate>
+      <plugin
+        filename="libignition-gazebo-diff-drive-system.so"
+        name="ignition::gazebo::systems::DiffDrive">
+        <topic>cmd_vel</topic>
+        <frame_id>odom</frame_id>
+        <child_frame_id>base_footprint</child_frame_id>
+      <!--    <odom_topic>odom</odom_topic> -->
+        <odom_topic>odom/unfiltered</odom_topic>
         <left_joint>left_wheel_joint</left_joint>
         <right_joint>right_wheel_joint</right_joint>
         <wheel_separation>${wheel_separation}</wheel_separation>
-        <wheel_diameter>${wheel_radius * 2}</wheel_diameter>
-        <max_wheel_acceleration>1.0</max_wheel_acceleration>
-        <robot_base_frame>base_footprint</robot_base_frame>
-        <publish_odom>true</publish_odom>
-        <publish_odom_tf>false</publish_odom_tf>
-        <publish_wheel_tf>true</publish_wheel_tf>
-        <odometry_frame>odom</odometry_frame>
+        <wheel_radius>${wheel_radius}</wheel_radius>
+        <odom_publish_frequency>20</odom_publish_frequency>
       </plugin>
+      <plugin
+        filename="ignition-gazebo-joint-state-publisher-system"
+        name="ignition::gazebo::systems::JointStatePublisher"/>
     </gazebo>
   </xacro:macro>

File: linorobot2_description/urdf/controllers/omni_drive.urdf.xacro (robot description, xacro)
@@ -1,17 +1,21 @@
 <robot xmlns:xacro="http://ros.org/wiki/xacro">
-  <xacro:macro name="omni_drive_controller">
+  <xacro:macro name="omni_drive_controller" params="wheel_separation wheel_base wheel_radius">
     <gazebo>
-    <plugin name="object_controller" filename="libgazebo_ros_planar_move.so">
-      <ros>
-        <remapping>odom:=odom/unfiltered</remapping>
-      </ros>
-      <command_topic>cmd_vel</command_topic>
-      <odometry_topic>odom/unfiltered</odometry_topic>
-      <odometry_frame>odom</odometry_frame>
-      <odometry_rate>20.0</odometry_rate>
-      <robot_base_frame>base_footprint</robot_base_frame>
-      <publish_odom>true</publish_odom>
-      <publish_odom_tf>false</publish_odom_tf>
-    </plugin>
+      <plugin
+        filename="ignition-gazebo-mecanum-drive-system"
+        name="ignition::gazebo::systems::MecanumDrive">
+        <topic>/cmd_vel</topic>
+        <frame_id>odom</frame_id>
+        <child_frame_id>base_footprint</child_frame_id>
+        <odom_topic>odom/unfiltered</odom_topic>
+        <front_left_joint>front_left_wheel_joint</front_left_joint>
+        <front_right_joint>front_right_wheel_joint</front_right_joint>
+        <back_left_joint>rear_left_wheel_joint</back_left_joint>
+        <back_right_joint>rear_right_wheel_joint</back_right_joint>
+        <wheel_separation>${wheel_separation}</wheel_separation>
+        <wheelbase>${wheel_base}</wheelbase>
+        <wheel_radius>${wheel_radius}</wheel_radius>
+        <odom_publish_frequency>50</odom_publish_frequency>
+      </plugin>
   </gazebo>
   </xacro:macro>

File: linorobot2_description/urdf/controllers/skid_steer.urdf.xacro (robot description, xacro)
@@ -1,10 +1,12 @@
 <robot xmlns:xacro="http://ros.org/wiki/xacro">
-  <xacro:macro name="diff_drive_controller" params="wheel_separation wheel_radius wheel_torque">
+  <xacro:macro name="diff_drive_controller" params="wheel_separation wheel_radius">
     <gazebo>
-      <plugin name="differential_drive_controller" filename="libgazebo_ros_diff_drive.so">
-        <ros>
-          <remapping>odom:=odom/unfiltered</remapping>
-        </ros>
-        <num_wheel_pairs>2</num_wheel_pairs>
+      <plugin
+        filename="ignition-gazebo-diff-drive-system"
+        name="ignition::gazebo::systems::DiffDrive">
+        <topic>/cmd_vel</topic>
+        <frame_id>odom</frame_id>
+        <child_frame_id>base_footprint</child_frame_id>
+        <odom_topic>odom/unfiltered</odom_topic>
         <left_joint>front_left_wheel_joint</left_joint>
         <right_joint>front_right_wheel_joint</right_joint>
@@ -12,14 +14,6 @@
         <right_joint>rear_right_wheel_joint</right_joint>
         <wheel_separation>${wheel_separation}</wheel_separation>
-        <wheel_separation>${wheel_separation}</wheel_separation>
-        <wheel_diameter>${wheel_radius * 2}</wheel_diameter>
-        <wheel_diameter>${wheel_radius * 2}</wheel_diameter>
-        <updateRate>100</updateRate>
-        <max_wheel_acceleration>1.0</max_wheel_acceleration>
-        <robot_base_frame>base_footprint</robot_base_frame>
-        <publish_odom>true</publish_odom>
-        <publish_odom_tf>false</publish_odom_tf>
-        <publish_wheel_tf>true</publish_wheel_tf>
-        <odometry_frame>odom</odometry_frame>
+        <wheel_radius>${wheel_radius}</wheel_radius>
+        <odom_publish_frequency>50</odom_publish_frequency>
       </plugin>
     </gazebo>

File: linorobot2_description/urdf/robots/2wd.urdf.xacro (robot description, xacro)
@@ -1,8 +1,10 @@
 <?xml version="1.0"?>
 <robot name="linorobot2_2wd" xmlns:xacro="http://ros.org/wiki/xacro">
+  <xacro:arg name="sim" default="false" />
   <xacro:include filename="$(find linorobot2_description)/urdf/2wd_properties.urdf.xacro" />
   <xacro:include filename="$(find linorobot2_description)/urdf/mech/base.urdf.xacro" />
   <xacro:include filename="$(find linorobot2_description)/urdf/mech/wheel.urdf.xacro" />
   <xacro:include filename="$(find linorobot2_description)/urdf/mech/caster_wheel.urdf.xacro" />
+  <xacro:include filename="$(find linorobot2_description)/urdf/sensors/plugins.urdf.xacro" />
   <xacro:include filename="$(find linorobot2_description)/urdf/sensors/imu.urdf.xacro" />
   <xacro:include filename="$(find linorobot2_description)/urdf/sensors/generic_laser.urdf.xacro" />
@@ -57,5 +59,5 @@
     <xacro:insert_block name="laser_pose" />
   </xacro:generic_laser>
-  <xacro:depth_sensor>
+  <xacro:depth_sensor sim="$(arg sim)" >
     <xacro:insert_block name="depth_sensor_pose" />
   </xacro:depth_sensor>
@@ -63,5 +65,4 @@
     wheel_separation="${wheel_pos_y * 2}"
     wheel_radius="${wheel_radius}"
-    wheel_torque="${wheel_torque}"
   />
 </robot>

File: linorobot2_description/urdf/robots/4wd.urdf.xacro (robot description, xacro)
@@ -1,7 +1,9 @@
 <?xml version="1.0"?>
 <robot name="linorobot2_2wd" xmlns:xacro="http://ros.org/wiki/xacro">
+  <xacro:arg name="sim" default="false" />
   <xacro:include filename="$(find linorobot2_description)/urdf/4wd_properties.urdf.xacro" />
   <xacro:include filename="$(find linorobot2_description)/urdf/mech/base.urdf.xacro" />
   <xacro:include filename="$(find linorobot2_description)/urdf/mech/wheel.urdf.xacro" />
+  <xacro:include filename="$(find linorobot2_description)/urdf/sensors/plugins.urdf.xacro" />
   <xacro:include filename="$(find linorobot2_description)/urdf/sensors/imu.urdf.xacro" />
   <xacro:include filename="$(find linorobot2_description)/urdf/sensors/generic_laser.urdf.xacro" />
@@ -56,5 +58,5 @@
     <xacro:insert_block name="laser_pose" />
   </xacro:generic_laser>
-  <xacro:depth_sensor>
+  <xacro:depth_sensor sim="$(arg sim)" >
     <xacro:insert_block name="depth_sensor_pose" />
   </xacro:depth_sensor>
@@ -62,5 +64,4 @@
     wheel_separation="${wheel_pos_y * 2}"
     wheel_radius="${wheel_radius}"
-    wheel_torque="${wheel_torque}"
   />
 </robot>

File: linorobot2_description/urdf/robots/mecanum.urdf.xacro (robot description, xacro)
@@ -1,7 +1,9 @@
 <?xml version="1.0"?>
 <robot name="linorobot2_2wd" xmlns:xacro="http://ros.org/wiki/xacro">
+  <xacro:arg name="sim" default="false" />
   <xacro:include filename="$(find linorobot2_description)/urdf/mecanum_properties.urdf.xacro" />
   <xacro:include filename="$(find linorobot2_description)/urdf/mech/base.urdf.xacro" />
   <xacro:include filename="$(find linorobot2_description)/urdf/mech/mecanum_wheel.urdf.xacro" />
+  <xacro:include filename="$(find linorobot2_description)/urdf/sensors/plugins.urdf.xacro" />
   <xacro:include filename="$(find linorobot2_description)/urdf/sensors/imu.urdf.xacro" />
   <xacro:include filename="$(find linorobot2_description)/urdf/sensors/generic_laser.urdf.xacro" />
@@ -56,7 +58,11 @@
     <xacro:insert_block name="laser_pose" />
   </xacro:generic_laser>
-  <xacro:depth_sensor>
+  <xacro:depth_sensor sim="$(arg sim)" >
     <xacro:insert_block name="depth_sensor_pose" />
   </xacro:depth_sensor>
-  <xacro:omni_drive_controller/>
+  <xacro:omni_drive_controller
+    wheel_separation="${wheel_pos_y * 2}"
+    wheel_base="${wheel_pos_x * 2}"
+    wheel_radius="${wheel_radius}"
+  />
 </robot>

File: linorobot2_description/urdf/robots/square.urdf.xacro (robot description, xacro)
@@ -1,15 +1,16 @@
 <?xml version="1.0"?>
 <robot name="linorobot2_2wd" xmlns:xacro="http://ros.org/wiki/xacro">
-  <xacro:property name="base_length" value="0.338" />
-  <xacro:property name="base_width" value="0.32" />
-  <xacro:property name="base_height" value="0.005" />
-  <xacro:property name="base_mass" value="5" />
-  <xacro:property name="wheel_radius" value="0.0675" />
-  <xacro:property name="wheel_width" value="0.022" />
-  <xacro:property name="wheel_pos_x" value="0.1015" />
-  <xacro:property name="wheel_pos_y" value="0.18" />
-  <xacro:property name="wheel_pos_z" value="-0.0125" />
+  <xacro:arg name="sim" default="false" />
+  <xacro:property name="base_length" value="0.25" />
+  <xacro:property name="base_width" value="0.25" />
+  <xacro:property name="base_height" value="0.003" />
+  <xacro:property name="base_mass" value="1" />
+  <xacro:property name="wheel_radius" value="0.045" />
+  <xacro:property name="wheel_width" value="0.01" />
+  <xacro:property name="wheel_pos_x" value="0.08" />
+  <xacro:property name="wheel_pos_y" value="0.12" />
+  <xacro:property name="wheel_pos_z" value="-0.045" />
   <xacro:property name="wheel_mass" value=".1" />
-  <xacro:property name="wheel_torque" value="40" />
+  <xacro:property name="wheel_torque" value="20" />
   <xacro:property name="front_caster_wheel" value="false" />
   <xacro:property name="rear_caster_wheel" value="true" />
@@ -22,11 +23,11 @@
   <xacro:include filename="$(find linorobot2_description)/urdf/controllers/diff_drive.urdf.xacro" />
   <xacro:property name="laser_pose">
-    <origin xyz="0.126 0 0.25" rpy="0 0 -0.78539816339"/>
+    <origin xyz="0.0 0 0.325" rpy="-3.1416 0 0"/>
   </xacro:property>
   <xacro:property name="base_laser_pose">
-    <origin xyz="0.179 0 -0.045" rpy="-3.1416 0 0"/>
+    <origin xyz="0.08 0 -0.05" rpy="-3.1416 0 0"/>
   </xacro:property>
   <xacro:property name="depth_sensor_pose">
-    <origin xyz="0.194 0.0 0.185" rpy="0 0 0"/>
+    <origin xyz="0.14 0.0 0.23" rpy="0 0 0"/>
   </xacro:property>
   <xacro:base
@@ -81,5 +82,5 @@
     <xacro:insert_block name="base_laser_pose" />
   </xacro:generic_base_laser>
-  <xacro:depth_sensor>
+  <xacro:depth_sensor sim="$(arg sim)" >
     <xacro:insert_block name="depth_sensor_pose" />
   </xacro:depth_sensor>
