Commit message: added camera properties

File: linorobot2_description/urdf/4wd_properties.urdf.xacro (robot description, xacro)
@@ -18,3 +18,6 @@
     <origin xyz="-0.065 0 0.255" rpy="0 0 0"/>
   </xacro:property>
+  <xacro:property name="rear_camera_sensor_pose">
+    <origin xyz="-0.2375 0.0 0.255" rpy="0 0 3.14159"/>
+  </xacro:property>
 </robot>

File: linorobot2_description/urdf/mecanum_properties.urdf.xacro (robot description, xacro)
@@ -18,3 +18,6 @@
     <origin xyz="0.2375 0 0.06" rpy="0 0 0"/>
   </xacro:property>
+  <xacro:property name="rear_camera_sensor_pose">
+    <origin xyz="-0.2375 0.0 0.06" rpy="0 0 3.14159"/>
+  </xacro:property>
 </robot>

File: linorobot2_description/urdf/robots/4wd.urdf.xacro (robot description, xacro)
@@ -7,4 +7,5 @@
   <xacro:include filename="$(find linorobot2_description)/urdf/sensors/generic_laser.urdf.xacro" />
   <xacro:include filename="$(find linorobot2_description)/urdf/sensors/depth_sensor.urdf.xacro" />
+  <xacro:include filename="$(find linorobot2_description)/urdf/sensors/camera.urdf.xacro" />
   <xacro:include filename="$(find linorobot2_description)/urdf/controllers/skid_steer.urdf.xacro" />
   <xacro:base
@@ -59,4 +60,10 @@
     <xacro:insert_block name="depth_sensor_pose" />
   </xacro:depth_sensor>
+  <xacro:rgb_camera
+      parent="base_link"
+      name="rear_rgb_camera"
+      topic_name="rear_rgb_camera/image">
+    <xacro:insert_block name="rear_camera_sensor_pose" />
+  </xacro:rgb_camera>
   <xacro:diff_drive_controller
     wheel_separation="${wheel_pos_y * 2}"

File: linorobot2_description/urdf/robots/mecanum.urdf.xacro (robot description, xacro)
@@ -7,4 +7,5 @@
   <xacro:include filename="$(find linorobot2_description)/urdf/sensors/generic_laser.urdf.xacro" />
   <xacro:include filename="$(find linorobot2_description)/urdf/sensors/depth_sensor.urdf.xacro" />
+  <xacro:include filename="$(find linorobot2_description)/urdf/sensors/camera.urdf.xacro" />
   <xacro:include filename="$(find linorobot2_description)/urdf/controllers/omni_drive.urdf.xacro" />
   <xacro:base
@@ -59,4 +60,10 @@
     <xacro:insert_block name="depth_sensor_pose" />
   </xacro:depth_sensor>
+  <xacro:rgb_camera
+      parent="base_link"
+      name="rear_rgb_camera"
+      topic_name="rear_rgb_camera/image">
+    <xacro:insert_block name="rear_camera_sensor_pose" />
+  </xacro:rgb_camera>
   <xacro:omni_drive_controller/>
 </robot>
