Commit message: added optical link, to address the tf issue while detecting apriltags

File: linorobot2_description/urdf/sensors/camera.urdf.xacro (robot description, xacro)
@@ -41,4 +41,10 @@
       <xacro:insert_block name="origin" />
     </joint>
+    <link name="${name}_optical_link"/>
+    <joint name="${name}_optical_joint" type="fixed">
+      <origin xyz="0 0 0" rpy="-1.57 0 -1.57"/>
+      <parent link="${name}_link"/>
+      <child link="${name}_optical_link"/>
+    </joint>
     <!-- https://github.com/ros-simulation/gazebo_ros_pkgs/wiki/ROS-2-Migration:-Camera#gazebo_ros_camera -->
     <gazebo reference="${name}_link">
@@ -59,5 +65,5 @@
           </ros>
           <hack_baseline>0.07</hack_baseline>
-          <frame_name>${name}_link</frame_name>
+          <frame_name>${name}_optical_link</frame_name>
           <distortion_k1>0.00000001</distortion_k1>
           <distortion_k2>0.00000001</distortion_k2>
